Commit message: Changed cmd_vel_topic to match the package name. Removed some comments

File: description/robot_core.xacro (robot description, xacro)
@@ -415,5 +415,5 @@
 <!-- Plugins -->
     <gazebo>
-        <plugin filename="libSimpleTrackedVehiclePlugin.so" name="tracked_vehicle">
+        <plugin filename="libSimpleTrackedVehiclePlugin.so" name="tracked_vehicle_plugin">
             <body>base_link</body>
             <left_track>left_track_link</left_track>
@@ -430,59 +430,7 @@
         <plugin filename="libKeysToCmdVelPlugin.so" name="keyboard_control">
             <publish_as_twist>true</publish_as_twist>
-            <cmd_vel_topic>~/tracked_vehicle/cmd_vel_twist</cmd_vel_topic>
+            <!-- This MUST be the name of the ros package -->
+            <cmd_vel_topic>~/tracked_robot/cmd_vel_twist</cmd_vel_topic>
         </plugin>
     </gazebo>
-<!--
-    <gazebo>
-        <plugin filename="ignition-gazebo-tracked-vehicle-system" name="gz::sim::systems::TrackedVehicle">
-            <left_track><link>left_track_link</link></left_track>
-            <left_track><link>rear_left_flipper_link</link></left_track>
-            <left_track><link>front_left_flipper_link</link></left_track>
-            <right_track><link>front_right_flipper_link</link></right_track>
-            <right_track><link>right_track_link</link></right_track>
-            <right_track><link>rear_right_flipper_link</link></right_track>
-            <tracks_separation>0.4</tracks_separation>
-            <tracks_height>0.18094</tracks_height>
-            <steering_efficiency>0.5</steering_efficiency>
-        </plugin>
-        <plugin filename="libignition-gazebo-track-controller-system.so" name="gz::sim::systems::TrackController">
-                <link>left_track_link</link>
-                <min_velocity>-1.0</min_velocity>
-                <max_velocity>1.0</max_velocity>
-        </plugin>
-        <plugin filename="libignition-gazebo-track-controller-system.so" name="gz::sim::systems::TrackController">
-                <link>right_track_link</link>
-                <min_velocity>-1.0</min_velocity>
-                <max_velocity>1.0</max_velocity>
-        </plugin>
-        <plugin filename="libignition-gazebo-track-controller-system.so" name="gz::sim::systems::TrackController">
-                <link>rear_left_flipper_link</link>
-                <min_velocity>-1.0</min_velocity>
-                <max_velocity>1.0</max_velocity>
-        </plugin>
-        <plugin filename="libignition-gazebo-track-controller-system.so" name="gz::sim::systems::TrackController">
-                <link>rear_right_flipper_link</link>
-                <min_velocity>-1.0</min_velocity>
-                <max_velocity>1.0</max_velocity>
-        </plugin>
-        <plugin filename="libignition-gazebo-track-controller-system.so" name="gz::sim::systems::TrackController">
-                <link>front_left_flipper_link</link>
-                <min_velocity>-1.0</min_velocity>
-                <max_velocity>1.0</max_velocity>
-        </plugin>
-        <plugin filename="libignition-gazebo-track-controller-system.so" name="gz::sim::systems::TrackController">
-                <link>front_right_flipper_link</link>
-                <min_velocity>-1.0</min_velocity>
-                <max_velocity>1.0</max_velocity>
-        </plugin>
-        <plugin filename="libignition-gazebo-triggered-publisher-system.so"
-                name="gz::sim::systems::TriggeredPublisher">
-            <input type="ignition.msgs.Int32" topic="/keyboard/keypress">
-                <match field="data">87</match>
-            </input>
-            <output type="ignition.msgs.Twist" topic="/model/my_bot/cmd_vel">
-                linear: {x: 1.0}, angular: {z: 0.0}
-            </output>
-        </plugin>
-    </gazebo>-->
 </robot>

Commit message: Updated mesh description location

File: description/robot_core.xacro (robot description, xacro)
@@ -73,5 +73,5 @@
             <material name="black"/>
             <geometry>
-                <mesh filename="$(find my_bot)/description/meshes/base_link.STL" />
+                <mesh filename="$(find tracked_robot)/description/meshes/base_link.STL" />
             </geometry>
         </visual>
@@ -101,5 +101,5 @@
             <material name="blue"/>
             <geometry>
-                <mesh filename="$(find my_bot)/description/meshes/left_track_link.STL" />
+                <mesh filename="$(find tracked_robot)/description/meshes/left_track_link.STL" />
             </geometry>
         </visual>
@@ -158,5 +158,5 @@
             <material name="blue"/>
             <geometry>
-                <mesh filename="$(find my_bot)/description/meshes/right_track_link.STL" />
+                <mesh filename="$(find tracked_robot)/description/meshes/right_track_link.STL" />
             </geometry>
         </visual>
@@ -214,5 +214,5 @@
             <material name="orange"/>
             <geometry>
-                <mesh filename="$(find my_bot)/description/meshes/back_left_fin_link.STL" />
+                <mesh filename="$(find tracked_robot)/description/meshes/back_left_fin_link.STL" />
             </geometry>
         </visual>
@@ -267,5 +267,5 @@
             <material name="black"/>
             <geometry>
-                <mesh filename="$(find my_bot)/description/meshes/back_right_fin_link.STL" />
+                <mesh filename="$(find tracked_robot)/description/meshes/back_right_fin_link.STL" />
             </geometry>
         </visual>
@@ -320,5 +320,5 @@
             <material name="orange"/>
             <geometry>
-                <mesh filename="$(find my_bot)/description/meshes/front_left_fin_link.STL" />
+                <mesh filename="$(find tracked_robot)/description/meshes/front_left_fin_link.STL" />
             </geometry>
         </visual>
@@ -373,5 +373,5 @@
             <origin xyz="0 ${flipper_visual_bias} 0" rpy="0 0 0" />
             <geometry>
-                <mesh filename="$(find my_bot)/description/meshes/front_right_fin_link.STL" />
+                <mesh filename="$(find tracked_robot)/description/meshes/front_right_fin_link.STL" />
             </geometry>
         </visual>

Commit message: Updated inertia values. These will need updating later

File: description/robot_core.xacro (robot description, xacro)
@@ -47,7 +47,7 @@
             <origin xyz="0 0 0" rpy="0 0 0" />
             <mass value="${base_mass}" />
-            <inertia ixx="0.203664" ixy="0" ixz="0"
-                iyy="0.136197" iyz="0"
-                izz="0.319921" />
+            <inertia ixx="5" ixy="0" ixz="0"
+                iyy="5" iyz="0"
+                izz="5" />
         </inertial>
         <collision name='base_collision_1'>
@@ -93,7 +93,7 @@
             <origin xyz="0 0 0" rpy="0 0 0" />
             <mass value="${track_mass}" />
-            <inertia ixx="0.15" ixy="0" ixz="0"
-                iyy="0.9" iyz="0"
-                izz="0.9" />
+            <inertia ixx="5" ixy="0" ixz="0"
+                iyy="5" iyz="0"
+                izz="5" />
         </inertial>
         <visual name='left_track_visual'>
@@ -150,7 +150,7 @@
             <origin xyz="0 0 0" rpy="0 0 0" />
             <mass value="${track_mass}" />
-            <inertia ixx="0.15" ixy="0" ixz="0"
-                iyy="0.9" iyz="0"
-                izz="0.9" />
+            <inertia ixx="5" ixy="0" ixz="0"
+                iyy="5" iyz="0"
+                izz="5" />
         </inertial>
         <visual name='right_track_visual'>
@@ -206,7 +206,7 @@
             <origin xyz="${-1*flipper_length/2} 0 0" rpy="0 0 0" />
             <mass value="${flipper_mass}" />
-            <inertia ixx="0.0025" ixy="0" ixz="0"
-                        iyy="0.022" iyz="0"
-                        izz="0.02" />
+            <inertia ixx="5" ixy="0" ixz="0"
+                iyy="5" iyz="0"
+                izz="5" />
         </inertial>
         <visual name='rear_left_flipper_visual'>
@@ -252,5 +252,5 @@
         <parent link="chassis_link" />
         <axis xyz="0 1 0" />
-        <limit lower="-3" upper="3" effort="-1" velocity="0.3" />
+        <limit lower="-3" upper="3" effort="1" velocity="1.0" />
     </joint>
     <!--rear_right_flipper -LINK-->
@@ -259,7 +259,7 @@
             <origin xyz="${-1*flipper_length/2} 0 0" rpy="0 0 0" />
             <mass value="${flipper_mass}" />
-            <inertia ixx="0.0025" ixy="0" ixz="0"
-                        iyy="0.022" iyz="0"
-                        izz="0.02" />
+            <inertia ixx="5" ixy="0" ixz="0"
+                iyy="5" iyz="0"
+                izz="5" />
         </inertial>
         <visual name='rear_right_flipper_visual'>
@@ -305,5 +305,5 @@
         <parent link="chassis_link" />
         <axis xyz="0 1 0" />
-        <limit lower="-3" upper="3" effort="-1" velocity="0.3" />
+        <limit lower="-3" upper="3" effort="1" velocity="1.0" />
     </joint>
     <!--front_left_flipper -LINK-->
@@ -312,7 +312,7 @@
             <origin xyz="${flipper_length/2} 0 0" rpy="0 0 0" />
             <mass value="${flipper_mass}" />
-            <inertia ixx="0.0025" ixy="0" ixz="0"
-                        iyy="0.022" iyz="0"
-                        izz="0.02" />
+            <inertia ixx="5" ixy="0" ixz="0"
+                iyy="5" iyz="0"
+                izz="5" />
         </inertial>
         <visual name='front_left_flipper_visual'>
@@ -358,5 +358,5 @@
         <parent link="chassis_link" />
         <axis xyz="0 1 0" />
-        <limit lower="-3" upper="3" effort="-1" velocity="0.3" />
+        <limit lower="-3" upper="3" effort="1" velocity="1.0" />
     </joint>
     <!--front_right_flipper - LINK-->
@@ -365,7 +365,7 @@
             <origin xyz="${flipper_length/2} 0 0" rpy="0 0 0" />
             <mass value="${flipper_mass}" />
-            <inertia ixx="0.0025" ixy="0" ixz="0"
-                        iyy="0.022" iyz="0"
-                        izz="0.02" />
+            <inertia ixx="5" ixy="0" ixz="0"
+                iyy="5" iyz="0"
+                izz="5" />
         </inertial>
         <visual name='front_right_flipper_link_visual'>
@@ -411,5 +411,5 @@
         <parent link="chassis_link" />
         <axis xyz="0 1 0" />
-        <limit lower="-3" upper="3" effort="-1" velocity="0.3" />
+        <limit lower="-3" upper="3" effort="1" velocity="1.0" />
     </joint>
 <!-- Plugins -->
@@ -434,3 +434,42 @@
         </plugin>
     </gazebo>
+    <ros2_control name="GazeboSystem" type="system">
+        <hardware>
+            <plugin>gazebo_ros2_control/GazeboSystem</plugin>
+        </hardware>
+    <joint name="front_right_flipper_joint">
+        <command_interface name="position">
+          <param name="min">-1</param>
+          <param name="max">1</param>
+        </command_interface>
+        <state_interface name="position"/>
+        <state_interface name="velocity"/>
+      </joint>
+      <joint name="front_left_flipper_joint">
+        <command_interface name="position">
+          <param name="min">-1</param>
+          <param name="max">1</param>
+        </command_interface>
+        <state_interface name="position"/>
+      </joint>
+      <joint name="rear_right_flipper_joint">
+        <command_interface name="position">
+          <param name="min">-1</param>
+          <param name="max">1</param>
+        </command_interface>
+        <state_interface name="position"/>
+      </joint>
+      <joint name="rear_left_flipper_joint">
+        <command_interface name="position">
+          <param name="min">-1</param>
+          <param name="max">1</param>
+        </command_interface>
+        <state_interface name="position"/>
+      </joint>
+    </ros2_control>
+    <gazebo>
+        <plugin filename="libgazebo_ros2_control.so" name="gazebo_ros2_control">
+            <parameters>$(find tracked_robot)/config/flipper_joint.yaml</parameters>
+        </plugin>
+    </gazebo>
 </robot>
